Commit message: commit

File: roomba/rviz/roomba.urdf.xacro (robot description, xacro)
@@ -19,4 +19,5 @@
         </xacro:inertial_cylinder>
     </link>
+    <link name="roomba/lidar/camera"></link>
     <link name="chassis">
         <visual>
@@ -90,4 +91,9 @@
         <origin xyz="0 0 0"/>
     </joint>
+    <joint name="camera_joint" type="fixed">
+        <parent link="roomba/lidar/gpu_lidar"/>
+        <child link="roomba/lidar/camera"/>
+        <origin xyz="0 0 0"/>
+    </joint>
     <joint name="left_wheel_joint" type="continuous">
         <parent link="chassis"/>
@@ -100,5 +106,5 @@
         <child link="right_wheel"/>
         <origin xyz="-0.35 -0.22 -0.065" rpy="1.5707 0 0"/>
-        <axis xyz="0 0 1"/>
+        <axis xyz="0 0 -1"/>
     </joint>
     <joint name="caster_wheel_joint" type="fixed">

Commit message: commit

File: roomba/rviz/roomba.urdf.xacro (robot description, xacro)
@@ -3,4 +3,5 @@
     <xacro:include filename="inertial_macros.xacro"/>
     <link name="base_link"></link>
+    <link name="base_footprint"></link>
     <link name="roomba/lidar/gpu_lidar">
         <visual>
@@ -84,4 +85,8 @@
     <joint name="base_joint" type="fixed">
         <parent link="base_link"/>
+        <child link="base_footprint"/>
+    </joint>
+    <joint name="base_joint" type="fixed">
+        <parent link="base_link"/>
         <child link="roomba/lidar/gpu_lidar"/>
     </joint>

Commit message: camera added and working

File: roomba/rviz/roomba.urdf.xacro (robot description, xacro)
@@ -3,5 +3,4 @@
     <xacro:include filename="inertial_macros.xacro"/>
     <link name="base_link"></link>
-    <link name="base_footprint"></link>
     <link name="roomba/lidar/gpu_lidar">
         <visual>
@@ -85,8 +84,4 @@
     <joint name="base_joint" type="fixed">
         <parent link="base_link"/>
-        <child link="base_footprint"/>
-    </joint>
-    <joint name="base_joint" type="fixed">
-        <parent link="base_link"/>
         <child link="roomba/lidar/gpu_lidar"/>
     </joint>
